File: Kicad/UPS.sch (KiCad schematic (older format))
At the start: 53 parts, among them J1 USB_B_Micro, J10 GET_UP_SERVO_RIGHT, J11 SPI, J12 I2C, J2 Conn_02x20_Odd_Even, J3 X_HEAD_PAN, J4 Y_HEAD_PAN, J5 X_CLAW, J6 Y_CLAW, J7 MOTOR_LEFT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

Commit message: Start add footprint
Parts:
- added J13: Conn_01x02_Male, symbol Connector:Conn_01x02_Male
- D1, D2, D3, D4, D5: footprint (none) -> LED_SMD:LED_0201_0603Metric
- J1: footprint (none) -> Connector_USB:USB_Micro-B_Amphenol_10103594-0001LF_Horizontal
- J10, J3, J4, J5, J6, J7, J8, J9: footprint (none) -> Connector_PinHeader_2.54mm:PinHeader_1x03_P2.54mm_Vertical
- J11: footprint (none) -> Connector_PinHeader_2.54mm:PinHeader_1x05_P2.54mm_Vertical
- J12: footprint (none) -> Connector_PinHeader_2.54mm:PinHeader_1x04_P2.54mm_Vertical
- J2: footprint (none) -> Connector_PinHeader_2.54mm:PinHeader_2x20_P2.54mm_Vertical
- SW1: footprint (none) -> Button_Switch_SMD:Panasonic_EVQPUJ_EVQPUA
Connections:
- net BATT+: no longer R2.1, R3.1
- net GND: now also U2.1 (CTG); no longer C3.2, C4.2, U2.9 (EP)
- new net: C3.2, C4.2, J13.2 (Pin_2), U2.9 (EP)
- new net: J13.1 (Pin_1), R2.1, R3.1
Other:
- moved on the sheet: C11
Changed lines of the file:
@@
 Wire Wire Line
 	2450 1450 2750 1450
-Wire Wire Line
-	2450 1450 1250 1450
-Connection ~ 2450 1450
-Wire Notes Line
-	750  1150 1300 1150
-Wire Notes Line
-	1300 1150 1300 2850
-Wire Notes Line
-	1300 2850 750  2850
-Wire Notes Line
-	750  2850 750  1150
 $Comp
 L eta1096:ETA1096 U3
@@
 F 0 "D2" V 1897 5878 50  0000 L CNN
 F 1 "LED" V 1988 5878 50  0000 L CNN
-F 2 "" H 1950 5800 50  0001 C CNN
+F 2 "LED_SMD:LED_0201_0603Metric" H 1950 5800 50  0001 C CNN
 F 3 "~" H 1950 5800 50  0001 C CNN
 	1    1950 5800
@@
 F 0 "D3" V 2289 5683 50  0000 R CNN
 F 1 "LED" V 2198 5683 50  0000 R CNN
-F 2 "" H 2250 5800 50  0001 C CNN
+F 2 "LED_SMD:LED_0201_0603Metric" H 2250 5800 50  0001 C CNN
 F 3 "~" H 2250 5800 50  0001 C CNN
 	1    2250 5800
@@
 F 0 "D4" H 2793 6016 50  0000 C CNN
 F 1 "LED" H 2793 5925 50  0000 C CNN
-F 2 "" H 2800 5800 50  0001 C CNN
+F 2 "LED_SMD:LED_0201_0603Metric" H 2800 5800 50  0001 C CNN
 F 3 "~" H 2800 5800 50  0001 C CNN
 	1    2800 5800
@@
 F 0 "SW1" H 5150 6435 50  0000 C CNN
 F 1 "SW_Push" H 5150 6344 50  0000 C CNN
-F 2 "" H 5150 6350 50  0001 C CNN
+F 2 "Button_Switch_SMD:Panasonic_EVQPUJ_EVQPUA" H 5150 6350 50  0001 C CNN
 F 3 "~" H 5150 6350 50  0001 C CNN
 	1    5150 6150
@@
 F 0 "D1" V 1639 5683 50  0000 R CNN
 F 1 "LED" V 1548 5683 50  0000 R CNN
-F 2 "" H 1600 5800 50  0001 C CNN
+F 2 "LED_SMD:LED_0201_0603Metric" H 1600 5800 50  0001 C CNN
 F 3 "~" H 1600 5800 50  0001 C CNN
 	1    1600 5800
@@
 F 0 "J1" H 807 5517 50  0000 C CNN
 F 1 "USB_B_Micro" H 807 5426 50  0000 C CNN
-F 2 "" H 900 5000 50  0001 C CNN
+F 2 "Connector_USB:USB_Micro-B_Amphenol_10103594-0001LF_Horizontal" H 900 5000 50  0001 C CNN
 F 3 "~" H 900 5000 50  0001 C CNN
 	1    750  5050
@@
 F 0 "D5" H 5093 5595 50  0000 C CNN
 F 1 "LED" H 5093 5686 50  0000 C CNN
-F 2 "" H 5100 5850 50  0001 C CNN
+F 2 "LED_SMD:LED_0201_0603Metric" H 5100 5850 50  0001 C CNN
 F 3 "~" H 5100 5850 50  0001 C CNN
 	1    5100 5850
@@
 U 1 1 5D624777
 P 7900 2000
-F 0 "L1" H 7900 2215 50  0000 C CNN
-F 1 "INDUCTOR" H 7900 2124 50  0000 C CNN
+F 0 "L1" H 7900 1900 50  0000 C CNN
+F 1 "INDUCTOR" H 7900 1950 50  0000 C CNN
 F 2 "" H 7900 2000 50  0001 C CNN
 F 3 "~" H 7900 2000 50  0001 C CNN
@@
 	-1   0    0    1
 $EndComp
-Wire Wire Line
-	7700 2100 8000 2100
 $Comp
 L Device:C C11
 U 1 1 5D62C104
-P 7700 2250
-F 0 "C11" H 7815 2296 50  0000 L CNN
-F 1 "10µf" H 7815 2205 50  0000 L CNN
-F 2 "" H 7738 2100 50  0001 C CNN
-F 3 "~" H 7700 2250 50  0001 C CNN
-	1    7700 2250
+P 7650 2250
+F 0 "C11" H 7400 2300 50  0000 L CNN
+F 1 "10µf" H 7400 2250 50  0000 L CNN
+F 2 "" H 7688 2100 50  0001 C CNN
+F 3 "~" H 7650 2250 50  0001 C CNN
+	1    7650 2250
 	1    0    0    -1
 $EndComp
@@
 U 1 1 5D62CA37
 P 8000 2250
-F 0 "C12" H 8115 2296 50  0000 L CNN
-F 1 "1µf" H 8115 2205 50  0000 L CNN
+F 0 "C12" H 8050 2300 50  0000 L CNN
+F 1 "1µf" H 8050 2250 50  0000 L CNN
 F 2 "" H 8038 2100 50  0001 C CNN
 F 3 "~" H 8000 2250 50  0001 C CNN
@@
 	4950 5450 5850 5450
 Connection ~ 5850 5450
-Text GLabel 7700 2900 3    50   Input ~ 0
+Text GLabel 7650 2900 3    50   Input ~ 0
 VIN
 Wire Wire Line
@@
 Wire Wire Line
 	7650 2000 7650 2100
-Wire Wire Line
-	7650 2100 7700 2100
-Connection ~ 7700 2100
 Text GLabel 8550 2400 2    50   Input ~ 0
 GND
@@
 NC
 Wire Wire Line
-	1250 2550 2450 2550
-Wire Wire Line
 	2450 2450 2450 2550
-Connection ~ 2450 2550
 Wire Wire Line
 	2450 2550 2750 2550
@@
 Connection ~ 2450 2150
 Wire Wire Line
-	7700 2900 7700 2400
+	7650 2900 7650 2400
 Text GLabel 6450 5150 2    50   Input ~ 0
 GND
 Text GLabel 7550 5450 2    50   Input ~ 0
 BATT+
-Text GLabel 1250 1450 0    50   Input ~ 0
+Text GLabel 1400 1950 0    50   Input ~ 0
 BATT+
-Text GLabel 1250 2550 0    50   Input ~ 0
+Text GLabel 1400 2050 0    50   Input ~ 0
 GND
 Text GLabel 5050 7250 0    50   Input ~ 0
@@
 F 0 "J2" H 6400 2917 50  0000 C CNN
 F 1 "Conn_02x20_Odd_Even" H 6400 2826 50  0000 C CNN
-F 2 "" H 6350 1800 50  0001 C CNN
+F 2 "Connector_PinHeader_2.54mm:PinHeader_2x20_P2.54mm_Vertical" H 6350 1800 50  0001 C CNN
 F 3 "~" H 6350 1800 50  0001 C CNN
 	1    6350 1800
@@
 F 0 "J6" H 10328 4876 50  0000 L CNN
 F 1 "Y_CLAW" H 10328 4785 50  0000 L CNN
-F 2 "" H 10300 4850 50  0001 C CNN
+F 2 "Connector_PinHeader_2.54mm:PinHeader_1x03_P2.54mm_Vertical" H 10300 4850 50  0001 C CNN
 F 3 "~" H 10300 4850 50  0001 C CNN
 	1    10300 4850
@@
 F 0 "J7" H 10328 5176 50  0000 L CNN
 F 1 "MOTOR_LEFT" H 10328 5085 50  0000 L CNN
-F 2 "" H 10300 5150 50  0001 C CNN
+F 2 "Connector_PinHeader_2.54mm:PinHeader_1x03_P2.54mm_Vertical" H 10300 5150 50  0001 C CNN
 F 3 "~" H 10300 5150 50  0001 C CNN
 	1    10300 5150
@@
 F 0 "J8" H 10328 5526 50  0000 L CNN
 F 1 "MOTOR_RIGHT" H 10328 5435 50  0000 L CNN
-F 2 "" H 10300 5500 50  0001 C CNN
+F 2 "Connector_PinHeader_2.54mm:PinHeader_1x03_P2.54mm_Vertical" H 10300 5500 50  0001 C CNN
 F 3 "~" H 10300 5500 50  0001 C CNN
 	1    10300 5500
@@
 F 0 "J9" H 10328 5876 50  0000 L CNN
 F 1 "GET_UP_SERVO_LEFT" H 10328 5785 50  0000 L CNN
-F 2 "" H 10300 5850 50  0001 C CNN
+F 2 "Connector_PinHeader_2.54mm:PinHeader_1x03_P2.54mm_Vertical" H 10300 5850 50  0001 C CNN
 F 3 "~" H 10300 5850 50  0001 C CNN
 	1    10300 5850
@@
 F 0 "J5" H 10328 4526 50  0000 L CNN
 F 1 "X_CLAW" H 10328 4435 50  0000 L CNN
-F 2 "" H 10300 4500 50  0001 C CNN
+F 2 "Connector_PinHeader_2.54mm:PinHeader_1x03_P2.54mm_Vertical" H 10300 4500 50  0001 C CNN
 F 3 "~" H 10300 4500 50  0001 C CNN
 	1    10300 4500
@@
 F 0 "J10" H 10328 6226 50  0000 L CNN
 F 1 "GET_UP_SERVO_RIGHT" H 10328 6135 50  0000 L CNN
-F 2 "" H 10300 6200 50  0001 C CNN
+F 2 "Connector_PinHeader_2.54mm:PinHeader_1x03_P2.54mm_Vertical" H 10300 6200 50  0001 C CNN
 F 3 "~" H 10300 6200 50  0001 C CNN
 	1    10300 6200
@@
 F 0 "J4" H 10328 4176 50  0000 L CNN
 F 1 "Y_HEAD_PAN" H 10328 4085 50  0000 L CNN
-F 2 "" H 10300 4150 50  0001 C CNN
+F 2 "Connector_PinHeader_2.54mm:PinHeader_1x03_P2.54mm_Vertical" H 10300 4150 50  0001 C CNN
 F 3 "~" H 10300 4150 50  0001 C CNN
 	1    10300 4150
@@
 F 0 "J3" H 10328 3826 50  0000 L CNN
 F 1 "X_HEAD_PAN" H 10328 3735 50  0000 L CNN
-F 2 "" H 10300 3800 50  0001 C CNN
+F 2 "Connector_PinHeader_2.54mm:PinHeader_1x03_P2.54mm_Vertical" H 10300 3800 50  0001 C CNN
 F 3 "~" H 10300 3800 50  0001 C CNN
 	1    10300 3800
@@
 F 0 "J11" H 9228 3926 50  0000 L CNN
 F 1 "SPI" H 9228 3835 50  0000 L CNN
-F 2 "" H 9200 3900 50  0001 C CNN
+F 2 "Connector_PinHeader_2.54mm:PinHeader_1x05_P2.54mm_Vertical" H 9200 3900 50  0001 C CNN
 F 3 "~" H 9200 3900 50  0001 C CNN
 	1    9200 3900
@@
 F 0 "J12" H 9228 4526 50  0000 L CNN
 F 1 "I2C" H 9228 4435 50  0000 L CNN
-F 2 "" H 9200 4550 50  0001 C CNN
+F 2 "Connector_PinHeader_2.54mm:PinHeader_1x04_P2.54mm_Vertical" H 9200 4550 50  0001 C CNN
 F 3 "~" H 9200 4550 50  0001 C CNN
 	1    9200 4550
@@
 Text GLabel 6450 4850 2    50   Output ~ 0
 +5V
+Connection ~ 7650 2100
+Wire Wire Line
+	7650 2100 8000 2100
+$Comp
+L Connector:Conn_01x02_Male J13
+U 1 1 5D63AEA3
+P 1400 1950
+F 0 "J13" H 1508 2131 50  0000 C CNN
+F 1 "Conn_01x02_Male" H 1508 2040 50  0000 C CNN
+F 2 "" H 1400 1950 50  0001 C CNN
+F 3 "~" H 1400 1950 50  0001 C CNN
+	1    1400 1950
+	1    0    0    -1
+$EndComp
+Connection ~ 2450 2550
+Wire Wire Line
+	2450 2550 1600 2550
+Wire Wire Line
+	1600 2550 1600 2050
+Wire Wire Line
+	1600 1950 2300 1950
+Wire Wire Line
+	2300 1950 2300 1450
+Wire Wire Line
+	2300 1450 2450 1450
+Connection ~ 2450 1450
+Text GLabel 3600 1950 0    50   Input ~ 0
+GND
 $EndSCHEMATC

Commit message: Minor change
Parts:
- removed J11: SPI, Connector_PinHeader_2.54mm:PinHeader_1x05_P2.54mm_Vertical, symbol Connector:Conn_01x05_Female
- removed J12: I2C, Connector_PinHeader_2.54mm:PinHeader_1x04_P2.54mm_Vertical, symbol Connector:Conn_01x04_Female
- J1: footprint Connector_USB:USB_Micro-B_Amphenol_10103594-0001LF_Horizontal -> Connector_USB:USB_Mini-B_Lumberg_2486_01_Horizontal
Connections:
- net +5V: now also C14.2
Other:
- moved on the sheet: D4, J10, J7, J8, J9
Changed lines of the file:
@@
 encoding utf-8
 Sheet 1 1
-Title ""
-Date ""
-Rev ""
-Comp ""
+Title "UPS"
+Date "2019-08-23"
+Rev "V1"
+Comp "DBI"
 Comment1 ""
 Comment2 ""
@@
 L Device:LED D4
 U 1 1 5D5ADF77
-P 2800 5800
-F 0 "D4" H 2793 6016 50  0000 C CNN
-F 1 "LED" H 2793 5925 50  0000 C CNN
-F 2 "LED_SMD:LED_0201_0603Metric" H 2800 5800 50  0001 C CNN
-F 3 "~" H 2800 5800 50  0001 C CNN
-	1    2800 5800
+P 2600 5800
+F 0 "D4" H 2593 6016 50  0000 C CNN
+F 1 "LED" H 2593 5925 50  0000 C CNN
+F 2 "LED_SMD:LED_0201_0603Metric" H 2600 5800 50  0001 C CNN
+F 3 "~" H 2600 5800 50  0001 C CNN
+	1    2600 5800
 	0    1    1    0
 $EndComp
@@
 Connection ~ 1950 5950
 Wire Wire Line
-	2250 5950 2800 5950
+	2250 5950 2600 5950
 Connection ~ 2250 5950
-Wire Wire Line
-	2250 5650 2800 5650
 Wire Wire Line
 	1600 5650 1600 5450
@@
 Wire Wire Line
 	1950 5450 3650 5450
-Wire Wire Line
-	2800 5950 3450 5950
-Wire Wire Line
-	3450 5950 3450 5650
-Wire Wire Line
-	3450 5650 3650 5650
-Connection ~ 2800 5950
-Wire Wire Line
-	3650 5550 2800 5550
-Wire Wire Line
-	2800 5550 2800 5650
-Connection ~ 2800 5650
 Wire Wire Line
 	4350 5650 4650 5650
@@
 F 0 "J1" H 807 5517 50  0000 C CNN
 F 1 "USB_B_Micro" H 807 5426 50  0000 C CNN
-F 2 "Connector_USB:USB_Micro-B_Amphenol_10103594-0001LF_Horizontal" H 900 5000 50  0001 C CNN
+F 2 "Connector_USB:USB_Mini-B_Lumberg_2486_01_Horizontal" H 900 5000 50  0001 C CNN
 F 3 "~" H 900 5000 50  0001 C CNN
 	1    750  5050
@@
 L Connector:Conn_01x03_Female J7
 U 1 1 5D649E24
-P 10300 5150
-F 0 "J7" H 10328 5176 50  0000 L CNN
-F 1 "MOTOR_LEFT" H 10328 5085 50  0000 L CNN
-F 2 "Connector_PinHeader_2.54mm:PinHeader_1x03_P2.54mm_Vertical" H 10300 5150 50  0001 C CNN
-F 3 "~" H 10300 5150 50  0001 C CNN
-	1    10300 5150
+P 10300 5200
+F 0 "J7" H 10328 5226 50  0000 L CNN
+F 1 "MOTOR_LEFT" H 10328 5135 50  0000 L CNN
+F 2 "Connector_PinHeader_2.54mm:PinHeader_1x03_P2.54mm_Vertical" H 10300 5200 50  0001 C CNN
+F 3 "~" H 10300 5200 50  0001 C CNN
+	1    10300 5200
 	1    0    0    -1
 $EndComp
@@
 L Connector:Conn_01x03_Female J8
 U 1 1 5D64A0D9
-P 10300 5500
-F 0 "J8" H 10328 5526 50  0000 L CNN
-F 1 "MOTOR_RIGHT" H 10328 5435 50  0000 L CNN
-F 2 "Connector_PinHeader_2.54mm:PinHeader_1x03_P2.54mm_Vertical" H 10300 5500 50  0001 C CNN
-F 3 "~" H 10300 5500 50  0001 C CNN
-	1    10300 5500
+P 10300 5550
+F 0 "J8" H 10328 5576 50  0000 L CNN
+F 1 "MOTOR_RIGHT" H 10328 5485 50  0000 L CNN
+F 2 "Connector_PinHeader_2.54mm:PinHeader_1x03_P2.54mm_Vertical" H 10300 5550 50  0001 C CNN
+F 3 "~" H 10300 5550 50  0001 C CNN
+	1    10300 5550
 	1    0    0    -1
 $EndComp
@@
 L Connector:Conn_01x03_Female J9
 U 1 1 5D64A47A
-P 10300 5850
-F 0 "J9" H 10328 5876 50  0000 L CNN
-F 1 "GET_UP_SERVO_LEFT" H 10328 5785 50  0000 L CNN
-F 2 "Connector_PinHeader_2.54mm:PinHeader_1x03_P2.54mm_Vertical" H 10300 5850 50  0001 C CNN
-F 3 "~" H 10300 5850 50  0001 C CNN
-	1    10300 5850
+P 10300 5900
+F 0 "J9" H 10328 5926 50  0000 L CNN
+F 1 "GET_UP_SERVO_LEFT" H 10328 5835 50  0000 L CNN
+F 2 "Connector_PinHeader_2.54mm:PinHeader_1x03_P2.54mm_Vertical" H 10300 5900 50  0001 C CNN
+F 3 "~" H 10300 5900 50  0001 C CNN
+	1    10300 5900
 	1    0    0    -1
 $EndComp
@@
 L Connector:Conn_01x03_Female J10
 U 1 1 5D64B5F4
-P 10300 6200
-F 0 "J10" H 10328 6226 50  0000 L CNN
-F 1 "GET_UP_SERVO_RIGHT" H 10328 6135 50  0000 L CNN
-F 2 "Connector_PinHeader_2.54mm:PinHeader_1x03_P2.54mm_Vertical" H 10300 6200 50  0001 C CNN
-F 3 "~" H 10300 6200 50  0001 C CNN
-	1    10300 6200
+P 10300 6250
+F 0 "J10" H 10328 6276 50  0000 L CNN
+F 1 "GET_UP_SERVO_RIGHT" H 10328 6185 50  0000 L CNN
+F 2 "Connector_PinHeader_2.54mm:PinHeader_1x03_P2.54mm_Vertical" H 10300 6250 50  0001 C CNN
+F 3 "~" H 10300 6250 50  0001 C CNN
+	1    10300 6250
 	1    0    0    -1
 $EndComp
@@
 Text GLabel 9750 4850 0    50   Input ~ 0
 +5V
-Text GLabel 9750 5150 0    50   Input ~ 0
-+5V
-Text GLabel 9750 5500 0    50   Input ~ 0
-+5V
-Text GLabel 9750 5850 0    50   Input ~ 0
-+5V
-Text GLabel 9750 6200 0    50   Input ~ 0
+Text GLabel 9750 5200 0    50   Input ~ 0
++5V
+Text GLabel 9750 5550 0    50   Input ~ 0
++5V
+Text GLabel 9750 5900 0    50   Input ~ 0
++5V
+Text GLabel 9750 6250 0    50   Input ~ 0
 +5V
 Text GLabel 9750 3900 0    50   Input ~ 0
@@
 Text GLabel 9750 4950 0    50   Input ~ 0
 GND
-Text GLabel 9750 5250 0    50   Input ~ 0
-GND
-Text GLabel 9750 5600 0    50   Input ~ 0
-GND
-Text GLabel 9750 5950 0    50   Input ~ 0
-GND
-Text GLabel 9750 6300 0    50   Input ~ 0
+Text GLabel 9750 5300 0    50   Input ~ 0
+GND
+Text GLabel 9750 5650 0    50   Input ~ 0
+GND
+Text GLabel 9750 6000 0    50   Input ~ 0
+GND
+Text GLabel 9750 6350 0    50   Input ~ 0
 GND
 Text GLabel 5500 6400 3    50   Input ~ 0
@@
 	9750 4950 10100 4950
 Wire Wire Line
-	9750 5150 10100 5150
-Wire Wire Line
-	9750 5250 10100 5250
-Wire Wire Line
-	9750 5500 10100 5500
-Wire Wire Line
-	9750 5850 10100 5850
-Wire Wire Line
-	10100 5600 9750 5600
-Wire Wire Line
-	9750 5950 10100 5950
-Wire Wire Line
-	9750 6200 10100 6200
-Wire Wire Line
-	9750 6300 10100 6300
+	9750 5200 10100 5200
+Wire Wire Line
+	9750 5300 10100 5300
+Wire Wire Line
+	9750 5550 10100 5550
+Wire Wire Line
+	9750 5900 10100 5900
+Wire Wire Line
+	10100 5650 9750 5650
+Wire Wire Line
+	9750 6000 10100 6000
+Wire Wire Line
+	9750 6250 10100 6250
+Wire Wire Line
+	9750 6350 10100 6350
 Text GLabel 9750 4400 0    50   Input ~ 0
 GPIO07
 Text GLabel 9750 4750 0    50   Input ~ 0
 GPIO08
-Text GLabel 9750 5050 0    50   Input ~ 0
+Text GLabel 9750 5100 0    50   Input ~ 0
 GPIO26
-Text GLabel 9750 5400 0    50   Input ~ 0
+Text GLabel 9750 5450 0    50   Input ~ 0
 GPIO27
 Wire Wire Line
@@
 	10100 4400 9750 4400
 Wire Wire Line
-	9750 5050 10100 5050
-Wire Wire Line
-	9750 5400 10100 5400
+	9750 5100 10100 5100
+Wire Wire Line
+	9750 5450 10100 5450
 Text GLabel 7650 2000 0    50   Input ~ 0
 VIN
 Text GLabel 3600 2250 0    50   Input ~ 0
 GND
-Text GLabel 9750 5750 0    50   Input ~ 0
+Text GLabel 9750 5800 0    50   Input ~ 0
 GPIO12
-Text GLabel 9750 6100 0    50   Input ~ 0
+Text GLabel 9750 6150 0    50   Input ~ 0
 GPIO13
 Wire Wire Line
-	10100 5750 9750 5750
-Wire Wire Line
-	10100 6100 9750 6100
-$Comp
-L Connector:Conn_01x05_Female J11
-U 1 1 5D700A91
-P 9200 3900
-F 0 "J11" H 9228 3926 50  0000 L CNN
-F 1 "SPI" H 9228 3835 50  0000 L CNN
-F 2 "Connector_PinHeader_2.54mm:PinHeader_1x05_P2.54mm_Vertical" H 9200 3900 50  0001 C CNN
-F 3 "~" H 9200 3900 50  0001 C CNN
-	1    9200 3900
-	1    0    0    -1
-$EndComp
-Text GLabel 8650 3800 0    50   Input ~ 0
-GPIO09
-Text GLabel 8650 3900 0    50   Input ~ 0
-GPIO10
-Text GLabel 8650 4000 0    50   Input ~ 0
-GPIO11
-Wire Wire Line
-	9000 3800 8650 3800
-Wire Wire Line
-	9000 3900 8650 3900
-Wire Wire Line
-	9000 4000 8650 4000
-$Comp
-L Connector:Conn_01x04_Female J12
-U 1 1 5D711701
-P 9200 4550
-F 0 "J12" H 9228 4526 50  0000 L CNN
-F 1 "I2C" H 9228 4435 50  0000 L CNN
-F 2 "Connector_PinHeader_2.54mm:PinHeader_1x04_P2.54mm_Vertical" H 9200 4550 50  0001 C CNN
-F 3 "~" H 9200 4550 50  0001 C CNN
-	1    9200 4550
-	1    0    0    -1
-$EndComp
-Text GLabel 8650 4650 0    50   Input ~ 0
-+3.3V
-Text GLabel 8650 4750 0    50   Input ~ 0
-GND
-Text GLabel 8650 4450 0    50   Input ~ 0
-GPIO02
-Text GLabel 8650 4550 0    50   Input ~ 0
-GPIO03
-Wire Wire Line
-	8650 4450 9000 4450
-Wire Wire Line
-	8650 4550 9000 4550
-Wire Wire Line
-	8650 4650 9000 4650
-Wire Wire Line
-	8650 4750 9000 4750
-Text GLabel 8650 3700 0    50   Input ~ 0
-+3.3V
-Text GLabel 8650 4100 0    50   Input ~ 0
-GND
-Wire Wire Line
-	8650 3700 9000 3700
-Wire Wire Line
-	8650 4100 9000 4100
+	10100 5800 9750 5800
+Wire Wire Line
+	10100 6150 9750 6150
 Text GLabel 6450 4850 2    50   Output ~ 0
 +5V
@@
 Text GLabel 3600 1950 0    50   Input ~ 0
 GND
+Wire Wire Line
+	2250 5550 2250 5650
+Wire Wire Line
+	2250 5550 2600 5550
+Wire Wire Line
+	2600 5650 2600 5550
+Connection ~ 2600 5550
+Wire Wire Line
+	2600 5550 3650 5550
+Wire Wire Line
+	2600 5950 2900 5950
+Wire Wire Line
+	2900 5950 2900 5650
+Wire Wire Line
+	2900 5650 3650 5650
+Connection ~ 2600 5950
+Text GLabel 10550 2650 3    50   Output ~ 0
++5V
 $EndSCHEMATC
