File: Kicad/UPS.sch (KiCad schematic (older format))
At the start: 52 parts, among them J1 USB_B_Micro, J10 GET_UP_SERVO_RIGHT, J13 Conn_01x02_Male, J2 Conn_02x20_Odd_Even, J3 X_HEAD_PAN, J4 Y_HEAD_PAN, J5 X_CLAW, J6 Y_CLAW, J7 MOTOR_LEFT, J8 MOTOR_RIGHT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

Commit message: Minor update
Parts:
- removed J7: MOTOR_LEFT, Connector_PinHeader_2.54mm:PinHeader_1x03_P2.54mm_Vertical, symbol Connector:Conn_01x03_Female
- removed J8: MOTOR_RIGHT, Connector_PinHeader_2.54mm:PinHeader_1x03_P2.54mm_Vertical, symbol Connector:Conn_01x03_Female
- added J? (x2): Conn_01x02_Female, symbol Connector:Conn_01x02_Female
Connections:
- net +5V: now also J?.1 (Pin_1), J?.1 (Pin_1)
- net GND: now also J?.2 (Pin_2), J?.2 (Pin_2)
Changed lines of the file:
@@
-$EndComp
-$Comp
-L Connector:Conn_01x03_Female J7
-U 1 1 5D649E24
-P 10300 5200
-F 0 "J7" H 10328 5226 50  0000 L CNN
-F 1 "MOTOR_LEFT" H 10328 5135 50  0000 L CNN
-F 2 "Connector_PinHeader_2.54mm:PinHeader_1x03_P2.54mm_Vertical" H 10300 5200 50  0001 C CNN
-F 3 "~" H 10300 5200 50  0001 C CNN
-	1    10300 5200
-	1    0    0    -1
-$EndComp
-$Comp
-L Connector:Conn_01x03_Female J8
-U 1 1 5D64A0D9
-P 10300 5550
-F 0 "J8" H 10328 5576 50  0000 L CNN
-F 1 "MOTOR_RIGHT" H 10328 5485 50  0000 L CNN
-F 2 "Connector_PinHeader_2.54mm:PinHeader_1x03_P2.54mm_Vertical" H 10300 5550 50  0001 C CNN
-F 3 "~" H 10300 5550 50  0001 C CNN
-	1    10300 5550
-	1    0    0    -1
 $EndComp
 $Comp
@@
 Text GLabel 10550 2650 3    50   Output ~ 0
 +5V
+$Comp
+L Connector:Conn_01x02_Female J?
+U 1 1 5D65A7C0
+P 10300 5200
+F 0 "J?" H 10328 5176 50  0000 L CNN
+F 1 "Conn_01x02_Female" H 10328 5085 50  0000 L CNN
+F 2 "" H 10300 5200 50  0001 C CNN
+F 3 "~" H 10300 5200 50  0001 C CNN
+	1    10300 5200
+	1    0    0    -1
+$EndComp
+$Comp
+L Connector:Conn_01x02_Female J?
+U 1 1 5D65B47C
+P 10300 5550
+F 0 "J?" H 10328 5526 50  0000 L CNN
+F 1 "Conn_01x02_Female" H 10328 5435 50  0000 L CNN
+F 2 "" H 10300 5550 50  0001 C CNN
+F 3 "~" H 10300 5550 50  0001 C CNN
+	1    10300 5550
+	1    0    0    -1
+$EndComp
 $EndSCHEMATC
