File: Kicad/UPS.kicad_pcb (KiCad board)
At the start: 2 copper layers, 18 parts, among them J1 USB_B_Micro, J10 GET_UP_SERVO_RIGHT, J11 SPI, J12 I2C, J2 Conn_02x20_Odd_Even, J3 X_HEAD_PAN, J4 Y_HEAD_PAN, J5 X_CLAW, J6 Y_CLAW, J7 MOTOR_LEFT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

Commit message: Minor change
Parts:
- removed J11: SPI, Connector_PinHeader_2.54mm:PinHeader_1x05_P2.54mm_Vertical
- removed J12: I2C, Connector_PinHeader_2.54mm:PinHeader_1x04_P2.54mm_Vertical
- moved J9 64.0 mm to (127.0, 86.4), turned to 90 degrees
- moved J5 58.5 mm to (127.0, 90.2), turned to 90 degrees
- moved J10 57.1 mm to (135.9, 86.4), turned to 90 degrees
- moved J7 52.3 mm to (144.8, 86.4), turned to 90 degrees
- moved J6 51.1 mm to (135.9, 90.2), turned to 90 degrees
- moved J8 50.3 mm to (153.7, 86.4), turned to 90 degrees
- moved J3 46.0 mm to (144.8, 90.2), turned to 90 degrees
- moved J4 44.0 mm to (153.7, 90.2), turned to 90 degrees
- moved D1 2.54 mm to (172.7, 83.8)
- moved D2 2.54 mm to (175.3, 83.8)
- moved D3 2.54 mm to (177.8, 83.8)
- moved D4 2.54 mm to (180.0, 83.8)
- moved SW1 2.54 mm to (185.4, 85.1)
- moved D5 1.27 mm to (190.5, 85.1)
Routing:
- net GND: track 0.00 -> 20.3 mm

Commit message: Minor update
Parts:
- moved J3 6.35 mm to (144.8, 96.5)
- moved J4 6.35 mm to (153.7, 96.5)
- moved J5 6.35 mm to (127.0, 96.5)
- moved J6 6.35 mm to (135.9, 96.5)
Changed lines of the file:
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@@
   )
   (module Connector_PinHeader_2.54mm:PinHeader_1x03_P2.54mm_Vertical (layer F.Cu)
-    (at 135.89 90.17 90)
+    (at 135.89 96.52 90)
     (descr "Through hole straight pin header, 1x03, 2.54mm pitch, single row")
     (tags "Through hole pin header THT 1x03 2.54mm single row")
@@
   )
   (module Connector_PinHeader_2.54mm:PinHeader_1x03_P2.54mm_Vertical (layer F.Cu)
-    (at 127 90.17 90)
+    (at 127 96.52 90)
     (descr "Through hole straight pin header, 1x03, 2.54mm pitch, single row")
     (tags "Through hole pin header THT 1x03 2.54mm single row")
@@
   )
   (module Connector_PinHeader_2.54mm:PinHeader_1x03_P2.54mm_Vertical (layer F.Cu)
-    (at 153.67 90.17 90)
+    (at 153.67 96.52 90)
     (descr "Through hole straight pin header, 1x03, 2.54mm pitch, single row")
     (tags "Through hole pin header THT 1x03 2.54mm single row")
@@
   )
   (module Connector_PinHeader_2.54mm:PinHeader_1x03_P2.54mm_Vertical (layer F.Cu)
-    (at 144.78 90.17 90)
+    (at 144.78 96.52 90)
     (descr "Through hole straight pin header, 1x03, 2.54mm pitch, single row")
     (tags "Through hole pin header THT 1x03 2.54mm single row")
